File: music-thing.sch (EAGLE design)
At the start: 6 parts

Commit message: finalize
Connections:
- net GND: now also U$1.GND1, U$2.GND, U$3.GND2; no longer U$3.GND1
Changed lines of the file:
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@@
 <part name="U$2" library="weller-eagle" deviceset="ASTAR32U4MINI" device=""/>
 <part name="CN1" library="adafruit" deviceset="DCBARREL" device="SMT"/>
-<part name="U$4" library="weller-eagle" deviceset="CON-MOTOR" device=""/>
 <part name="C1" library="SparkFun-Capacitors" deviceset="100UF-63V-20%(ELECT)" device="" value="100uF"/>
 <part name="U$3" library="weller-eagle" deviceset="CON-USB-READER-V18" device=""/>
+<part name="U$4" library="weller-eagle" deviceset="CON-MOTOR" device=""/>
 </parts>
 <sheets>
@@
 <instance part="U$2" gate="G$1" x="38.1" y="63.5"/>
 <instance part="CN1" gate="G$1" x="88.9" y="73.66" rot="R180"/>
-<instance part="U$4" gate="G$1" x="134.62" y="10.16"/>
 <instance part="C1" gate="G$1" x="68.58" y="76.2" rot="R180"/>
 <instance part="U$3" gate="G$1" x="17.78" y="33.02" rot="R180"/>
+<instance part="U$4" gate="G$1" x="132.08" y="10.16"/>
 </instances>
 <busses>
 </busses>
 <nets>
-<net name="N$3" class="0">
-<segment>
-<pinref part="U$1" gate="G$1" pin="1A"/>
-<pinref part="U$4" gate="G$1" pin="B1"/>
-<wire x1="129.54" y1="20.32" x2="111.76" y2="20.32" width="0.1524" layer="91"/>
-</segment>
-</net>
-<net name="N$4" class="0">
-<segment>
-<pinref part="U$1" gate="G$1" pin="1B"/>
-<pinref part="U$4" gate="G$1" pin="B2"/>
-<wire x1="129.54" y1="15.24" x2="111.76" y2="15.24" width="0.1524" layer="91"/>
-</segment>
-</net>
 <net name="5V" class="0">
 <segment>
@@
 <pinref part="U$3" gate="G$1" pin="VCC"/>
 <wire x1="17.78" y1="-5.08" x2="22.86" y2="-5.08" width="0.1524" layer="91"/>
+<label x="20.32" y="-5.08" size="1.778" layer="95"/>
 </segment>
 </net>
 <net name="GND" class="0">
-<segment>
-<wire x1="109.22" y1="35.56" x2="114.3" y2="35.56" width="0.1524" layer="91"/>
-<label x="109.22" y="35.56" size="1.778" layer="95"/>
-</segment>
-<segment>
-<wire x1="109.22" y1="5.08" x2="114.3" y2="5.08" width="0.1524" layer="91"/>
-<label x="109.22" y="5.08" size="1.778" layer="95"/>
-</segment>
-<segment>
-<wire x1="35.56" y1="81.28" x2="27.94" y2="81.28" width="0.1524" layer="91"/>
-<label x="27.94" y="81.28" size="1.778" layer="95"/>
-</segment>
-<segment>
-<wire x1="55.88" y1="66.04" x2="60.96" y2="66.04" width="0.1524" layer="91"/>
-<label x="55.88" y="66.04" size="1.778" layer="95"/>
-</segment>
 <segment>
 <pinref part="CN1" gate="G$1" pin="GNDBREAK"/>
@@
 </segment>
 <segment>
-<pinref part="U$3" gate="G$1" pin="GND1"/>
-<wire x1="17.78" y1="0" x2="22.86" y2="0" width="0.1524" layer="91"/>
+<pinref part="U$3" gate="G$1" pin="GND2"/>
+<wire x1="17.78" y1="30.48" x2="22.86" y2="30.48" width="0.1524" layer="91"/>
+<label x="17.78" y="30.48" size="1.778" layer="95"/>
 </segment>
-</net>
-<net name="N$2" class="0">
 <segment>
-<pinref part="U$1" gate="G$1" pin="2A"/>
-<pinref part="U$4" gate="G$1" pin="A2"/>
-<wire x1="111.76" y1="25.4" x2="129.54" y2="25.4" width="0.1524" layer="91"/>
+<pinref part="U$1" gate="G$1" pin="GND1"/>
+<wire x1="111.76" y1="35.56" x2="119.38" y2="35.56" width="0.1524" layer="91"/>
+<label x="114.3" y="35.56" size="1.778" layer="95"/>
 </segment>
-</net>
-<net name="N$1" class="0">
 <segment>
-<pinref part="U$1" gate="G$1" pin="2B"/>
-<pinref part="U$4" gate="G$1" pin="A1"/>
-<wire x1="111.76" y1="30.48" x2="129.54" y2="30.48" width="0.1524" layer="91"/>
+<pinref part="U$2" gate="G$1" pin="GND"/>
+<wire x1="58.42" y1="66.04" x2="68.58" y2="66.04" width="0.1524" layer="91"/>
+<label x="60.96" y="66.04" size="1.778" layer="95"/>
 </segment>
 </net>
@@
 </segment>
 </net>
+<net name="N$1" class="0">
+<segment>
+<pinref part="U$1" gate="G$1" pin="2B"/>
+<pinref part="U$4" gate="G$1" pin="A1"/>
+<wire x1="111.76" y1="30.48" x2="127" y2="30.48" width="0.1524" layer="91"/>
+</segment>
+</net>
+<net name="N$2" class="0">
+<segment>
+<pinref part="U$1" gate="G$1" pin="2A"/>
+<pinref part="U$4" gate="G$1" pin="A2"/>
+<wire x1="111.76" y1="25.4" x2="127" y2="25.4" width="0.1524" layer="91"/>
+</segment>
+</net>
+<net name="N$3" class="0">
+<segment>
+<pinref part="U$1" gate="G$1" pin="1A"/>
+<pinref part="U$4" gate="G$1" pin="B1"/>
+<wire x1="111.76" y1="20.32" x2="127" y2="20.32" width="0.1524" layer="91"/>
+</segment>
+</net>
+<net name="N$4" class="0">
+<segment>
+<pinref part="U$1" gate="G$1" pin="1B"/>
+<pinref part="U$4" gate="G$1" pin="B2"/>
+<wire x1="111.76" y1="15.24" x2="127" y2="15.24" width="0.1524" layer="91"/>
+</segment>
+</net>

Commit message: new layout
Parts:
- removed C1: 100uF, SparkFun-Capacitors:100UF-63V-20%(ELECT)
Connections:
- removed net N$5: C1.+, CN1.PWR, U$1.VMOT, U$2.VIN
- new net N$16: CN1.PWR, U$1.VMOT, U$2.VIN
- net GND: now also U$2.GND2; no longer C1.-, U$2.GND
Changed lines of the file:
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@@
 <part name="U$2" library="weller-eagle" deviceset="ASTAR32U4MINI" device=""/>
 <part name="CN1" library="adafruit" deviceset="DCBARREL" device="SMT"/>
-<part name="C1" library="SparkFun-Capacitors" deviceset="100UF-63V-20%(ELECT)" device="" value="100uF"/>
 <part name="U$3" library="weller-eagle" deviceset="CON-USB-READER-V18" device=""/>
 <part name="U$4" library="weller-eagle" deviceset="CON-MOTOR" device=""/>
@@
 <instance part="U$2" gate="G$1" x="38.1" y="63.5"/>
 <instance part="CN1" gate="G$1" x="88.9" y="73.66" rot="R180"/>
-<instance part="C1" gate="G$1" x="68.58" y="76.2" rot="R180"/>
 <instance part="U$3" gate="G$1" x="17.78" y="33.02" rot="R180"/>
 <instance part="U$4" gate="G$1" x="132.08" y="10.16"/>
@@
 <wire x1="86.36" y1="76.2" x2="76.2" y2="76.2" width="0.1524" layer="91"/>
 <label x="76.2" y="78.74" size="1.778" layer="95"/>
-<pinref part="C1" gate="G$1" pin="-"/>
-<wire x1="68.58" y1="81.28" x2="76.2" y2="81.28" width="0.1524" layer="91"/>
-<wire x1="76.2" y1="81.28" x2="76.2" y2="76.2" width="0.1524" layer="91"/>
 </segment>
 <segment>
@@
 </segment>
 <segment>
-<pinref part="U$2" gate="G$1" pin="GND"/>
+<pinref part="U$2" gate="G$1" pin="GND2"/>
 <wire x1="58.42" y1="66.04" x2="68.58" y2="66.04" width="0.1524" layer="91"/>
 <label x="60.96" y="66.04" size="1.778" layer="95"/>
@@
 </segment>
 </net>
-<net name="N$5" class="0">
+<net name="N$16" class="0">
 <segment>
 <pinref part="CN1" gate="G$1" pin="PWR"/>
 <pinref part="U$2" gate="G$1" pin="VIN"/>
-<wire x1="86.36" y1="71.12" x2="68.58" y2="71.12" width="0.1524" layer="91"/>
+<wire x1="86.36" y1="71.12" x2="58.42" y2="71.12" width="0.1524" layer="91"/>
 <pinref part="U$1" gate="G$1" pin="VMOT"/>
-<wire x1="68.58" y1="71.12" x2="58.42" y2="71.12" width="0.1524" layer="91"/>
 <wire x1="111.76" y1="40.64" x2="111.76" y2="66.04" width="0.1524" layer="91"/>
 <wire x1="111.76" y1="66.04" x2="86.36" y2="66.04" width="0.1524" layer="91"/>
 <wire x1="86.36" y1="66.04" x2="86.36" y2="71.12" width="0.1524" layer="91"/>
 <junction x="86.36" y="71.12"/>
-<pinref part="C1" gate="G$1" pin="+"/>
-<wire x1="68.58" y1="73.66" x2="68.58" y2="71.12" width="0.1524" layer="91"/>
-<junction x="68.58" y="71.12"/>
 </segment>
 </net>
